Commit message: Add Chunk 3: Gazebo Harmonic simulation with diff-drive ros2_control

File: surveillance_robot_ws/src/surveillance_robot_description/urdf/robot.urdf.xacro (robot description, xacro)
@@ -4,8 +4,24 @@
   This file only wires the modular pieces together in the correct order:
     dimensions  -> materials -> inertial macros -> chassis -> wheels -> sensors
+    -> (simulation-only) ros2_control + gazebo
   Ordering matters: properties and macros must be defined before the files that
   consume them. No geometry or dimensions are declared here directly.
+  Simulation gating:
+  sim_mode (arg, default false):
+      false -> pure kinematic description (Chunk 2 behaviour, RViz/xacro only).
+               No ros2_control, no Gazebo plugins. Fully backward compatible.
+      true  -> also pull in the ros2_control hardware block and the gz-sim
+               plugins so the model can be spawned and driven in Gazebo.
+  controllers_file (arg):
+      Absolute path to the ros2_control YAML handed to the gz_ros2_control
+      plugin. Defaults to the installed surveillance_robot_gazebo config so the
+      description stays reusable but works out-of-the-box under simulation.
 -->
 <robot xmlns:xacro="http://www.ros.org/wiki/xacro" name="surveillance_robot">
+  <!-- Simulation switches. -->
+  <xacro:arg name="sim_mode" default="false"/>
+  <xacro:arg name="controllers_file"
+             default="$(find surveillance_robot_gazebo)/config/controllers.yaml"/>
+  <xacro:property name="sim_mode" value="$(arg sim_mode)"/>
   <!-- Parameters and reusable building blocks (must come first). -->
   <xacro:include filename="$(find surveillance_robot_description)/urdf/dimensions.xacro"/>
@@ -17,3 +33,10 @@
   <!-- Structural sensor mounting frames (no sensors attached yet). -->
   <xacro:include filename="$(find surveillance_robot_description)/urdf/sensors.xacro"/>
+  <!-- Simulation-only: ros2_control interfaces + Gazebo plugins/friction. -->
+  <xacro:if value="${sim_mode}">
+    <xacro:include filename="$(find surveillance_robot_description)/urdf/ros2_control.xacro"/>
+    <xacro:include filename="$(find surveillance_robot_description)/urdf/gazebo.xacro"/>
+    <xacro:diff_drive_ros2_control/>
+    <xacro:gazebo_sim controllers_file="$(arg controllers_file)"/>
+  </xacro:if>
 </robot>

Commit message: feat: enhance robot URDF and add new sensor configurations
Added camera optical frame and updated sensor mounting frames. Included Gazebo sensor configurations and dependencies.

Co-authored-by: mayureshcode <148183189+mayureshcode@users.noreply.github.com>

File: surveillance_robot_ws/src/surveillance_robot_description/urdf/robot.urdf.xacro (robot description, xacro)
@@ -31,5 +31,5 @@
   <xacro:include filename="$(find surveillance_robot_description)/urdf/chassis.xacro"/>
   <xacro:include filename="$(find surveillance_robot_description)/urdf/wheels.xacro"/>
-  <!-- Structural sensor mounting frames (no sensors attached yet). -->
+  <!-- Structural sensor mounting frames, including the camera optical frame. -->
   <xacro:include filename="$(find surveillance_robot_description)/urdf/sensors.xacro"/>
   <!-- Simulation-only: ros2_control interfaces + Gazebo plugins/friction. -->
@@ -37,6 +37,10 @@
     <xacro:include filename="$(find surveillance_robot_description)/urdf/ros2_control.xacro"/>
     <xacro:include filename="$(find surveillance_robot_description)/urdf/gazebo.xacro"/>
+    <xacro:include filename="$(find surveillance_robot_gazebo)/urdf/gazebo_sensors.xacro"/>
+    <xacro:arg name="sensors_file"
+               default="$(find surveillance_robot_gazebo)/config/sensors.yaml"/>
     <xacro:diff_drive_ros2_control/>
     <xacro:gazebo_sim controllers_file="$(arg controllers_file)"/>
+    <xacro:gazebo_sensors config_file="$(arg sensors_file)"/>
   </xacro:if>
 </robot>

File: surveillance_robot_ws/src/surveillance_robot_description/urdf/sensors.xacro (robot description, xacro)
@@ -1,12 +1,11 @@
 <?xml version="1.0"?>
 <!--
-  STRUCTURAL sensor mounting frames only. No Gazebo sensors, no plugins, no
-  data topics yet. Chunk 4 will attach the actual LiDAR / camera / IMU to these
-  frames.
+  STRUCTURAL sensor mounting frames only. Gazebo sensors and topic configuration
+  live separately in surveillance_robot_gazebo/urdf/gazebo_sensors.xacro and are
+  attached only when sim_mode is enabled.
   Frame conventions (REP 103): x = forward, y = left, z = up.
   laser_link  : upright, axes aligned with base_link (LiDAR scans in its xy).
-  camera_link : mounting frame aligned with base_link, +x forward. The optical
-                frame (z-forward, x-right) is intentionally NOT created here;
-                it belongs with the camera sensor in Chunk 4.
+  camera_link : mounting frame aligned with base_link, +x forward. Its optical
+                child uses z-forward, x-right, y-down for ROS camera messages.
   imu_link    : aligned with base_link.
   Small visual markers are included purely so the mounts are visible in RViz.
@@ -61,4 +60,12 @@
     </xacro:inertial_box>
   </link>
+  <!-- The optical origin is co-located with the mount: +z forward, +x right,
+       +y down. robot_state_publisher is the only publisher of this fixed TF. -->
+  <joint name="camera_optical_joint" type="fixed">
+    <parent link="camera_link"/>
+    <child link="camera_optical_frame"/>
+    <origin xyz="0 0 0" rpy="${-PI_2} 0 ${-PI_2}"/>
+  </joint>
+  <link name="camera_optical_frame"/>
   <!-- ================= IMU mount ================= -->
   <joint name="imu_joint" type="fixed">
